File: A4988_Pmod.kicad_pcb (KiCad board)
At the start: 2 copper layers, 47.2 x 24.4 mm, 6 parts, among them J1 Pmod_male, J2 Screw_Terminal_01x04, J3 Jack-DC, J4 Screw_Terminal_01x02, U1 A4988_MODULE

Commit message: 2
Connections:
- J3 pad 3: (no net) -> GND
Routing:
- net /STEP: track 22.8 -> 24.0 mm
- net GND: vias 8 -> 9
Other:
- board text added: "Pmod A4988 Ver 0.2"
- board text removed: "Pmod A4988 Ver 0.1"
Changed lines of the file:
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@@
     (pad "2" thru_hole roundrect (at -6 0 90) (size 3 3.5) (drill oval 1 3) (layers *.Cu *.Mask) (roundrect_rratio 0.25)
       (net 6 "GND") (pintype "passive"))
-    (pad "3" thru_hole circle (at -3 4.7 90) (size 2.5 2.5) (drill oval 2.4 0.8) (layers *.Cu *.Mask))
+    (pad "3" thru_hole circle (at -3 4.7 90) (size 2.5 2.5) (drill oval 2.4 0.8) (layers *.Cu *.Mask)
+      (net 6 "GND"))
     (model "${KICAD6_3DMODEL_DIR}/Connector_BarrelJack.3dshapes/BarrelJack_Horizontal.wrl"
       (offset (xyz 0 0 0))
@@
     (effects (font (size 1 1) (thickness 0.15)) (justify mirror))
   )
-  (gr_text "Pmod A4988 Ver 0.1" (at 138.938 73.152) (layer "F.SilkS")
+  (gr_text "Pmod A4988 Ver 0.2" (at 138.938 73.152) (layer "F.SilkS")
     (effects (font (size 1 1) (thickness 0.15)))
   )
@@
   (segment (start 123.932 75.428) (end 125.212 75.428) (width 0.25) (layer "F.Cu") (net 2))
   (segment (start 126.746 76.962) (end 126.746 86.614) (width 0.25) (layer "F.Cu") (net 2))
-  (segment (start 119.37 90.668) (end 116.84 88.138) (width 0.25) (layer "F.Cu") (net 3))
-  (segment (start 116.84 88.138) (end 113.284 88.138) (width 0.25) (layer "F.Cu") (net 3))
-  (segment (start 107.696 80.264) (end 106.742 80.264) (width 0.25) (layer "F.Cu") (net 3))
-  (segment (start 112.268 84.836) (end 107.696 80.264) (width 0.25) (layer "F.Cu") (net 3))
   (segment (start 123.932 90.668) (end 119.37 90.668) (width 0.25) (layer "F.Cu") (net 3))
-  (segment (start 112.268 87.122) (end 112.268 84.836) (width 0.25) (layer "F.Cu") (net 3))
-  (segment (start 113.284 88.138) (end 112.268 87.122) (width 0.25) (layer "F.Cu") (net 3))
+  (segment (start 116.967 88.265) (end 112.776 88.265) (width 0.25) (layer "F.Cu") (net 3))
+  (segment (start 112.268 87.757) (end 112.268 83.439) (width 0.25) (layer "F.Cu") (net 3))
+  (segment (start 119.37 90.668) (end 116.967 88.265) (width 0.25) (layer "F.Cu") (net 3))
+  (segment (start 109.093 80.264) (end 106.742 80.264) (width 0.25) (layer "F.Cu") (net 3))
+  (segment (start 112.776 88.265) (end 112.268 87.757) (width 0.25) (layer "F.Cu") (net 3))
+  (segment (start 112.268 83.439) (end 109.093 80.264) (width 0.25) (layer "F.Cu") (net 3))
+  (segment (start 112.268 94.742) (end 125.476 94.742) (width 0.25) (layer "F.Cu") (net 4))
+  (segment (start 106.742 85.344) (end 107.823 85.344) (width 0.25) (layer "F.Cu") (net 4))
+  (segment (start 109.093 86.614) (end 109.093 91.567) (width 0.25) (layer "F.Cu") (net 4))
+  (segment (start 107.823 85.344) (end 109.093 86.614) (width 0.25) (layer "F.Cu") (net 4))
+  (segment (start 109.093 91.567) (end 112.268 94.742) (width 0.25) (layer "F.Cu") (net 4))
+  (segment (start 125.476 94.742) (end 126.746 93.472) (width 0.25) (layer "F.Cu") (net 4))
+  (segment (start 125.466 88.128) (end 123.932 88.128) (width 0.25) (layer "F.Cu") (net 4))
+  (segment (start 126.746 93.472) (end 126.746 89.408) (width 0.25) (layer "F.Cu") (net 4))
   (segment (start 126.746 89.408) (end 125.466 88.128) (width 0.25) (layer "F.Cu") (net 4))
-  (segment (start 108.204 85.344) (end 109.22 86.36) (width 0.25) (layer "F.Cu") (net 4))
-  (segment (start 125.466 88.128) (end 123.932 88.128) (width 0.25) (layer "F.Cu") (net 4))
-  (segment (start 109.22 86.36) (end 109.22 91.694) (width 0.25) (layer "F.Cu") (net 4))
-  (segment (start 106.742 85.344) (end 108.204 85.344) (width 0.25) (layer "F.Cu") (net 4))
-  (segment (start 112.268 94.742) (end 125.476 94.742) (width 0.25) (layer "F.Cu") (net 4))
-  (segment (start 126.746 93.472) (end 126.746 89.408) (width 0.25) (layer "F.Cu") (net 4))
-  (segment (start 125.476 94.742) (end 126.746 93.472) (width 0.25) (layer "F.Cu") (net 4))
-  (segment (start 109.22 91.694) (end 112.268 94.742) (width 0.25) (layer "F.Cu") (net 4))
-  (segment (start 110.236 90.678) (end 110.236 85.09) (width 0.25) (layer "F.Cu") (net 5))
-  (segment (start 110.236 85.09) (end 107.95 82.804) (width 0.25) (layer "F.Cu") (net 5))
-  (segment (start 113.284 93.726) (end 110.236 90.678) (width 0.25) (layer "F.Cu") (net 5))
+  (segment (start 107.061 82.804) (end 106.742 82.804) (width 0.25) (layer "F.Cu") (net 5))
   (segment (start 123.932 93.208) (end 123.414 93.726) (width 0.25) (layer "F.Cu") (net 5))
-  (segment (start 123.414 93.726) (end 113.284 93.726) (width 0.25) (layer "F.Cu") (net 5))
-  (segment (start 107.95 82.804) (end 106.742 82.804) (width 0.25) (layer "F.Cu") (net 5))
+  (segment (start 109.982 90.678) (end 109.982 85.725) (width 0.25) (layer "F.Cu") (net 5))
+  (segment (start 123.414 93.726) (end 113.03 93.726) (width 0.25) (layer "F.Cu") (net 5))
+  (segment (start 113.03 93.726) (end 109.982 90.678) (width 0.25) (layer "F.Cu") (net 5))
+  (segment (start 109.982 85.725) (end 107.061 82.804) (width 0.25) (layer "F.Cu") (net 5))
+  (via (at 109.728 83.058) (size 0.8) (drill 0.4) (layers "F.Cu" "B.Cu") (free) (net 6))
   (via (at 108.966 73.66) (size 0.8) (drill 0.4) (layers "F.Cu" "B.Cu") (free) (net 6))
   (via (at 106.426 94.234) (size 0.8) (drill 0.4) (layers "F.Cu" "B.Cu") (free) (net 6))
-  (via (at 112.522 83.058) (size 0.8) (drill 0.4) (layers "F.Cu" "B.Cu") (free) (net 6))
+  (via (at 113.284 82.423) (size 0.8) (drill 0.4) (layers "F.Cu" "B.Cu") (free) (net 6))
   (via (at 101.6 81.534) (size 0.8) (drill 0.4) (layers "F.Cu" "B.Cu") (free) (net 6))
-  (via (at 119.38 91.948) (size 0.8) (drill 0.4) (layers "F.Cu" "B.Cu") (free) (net 6))
-  (via (at 120.396 83.312) (size 0.8) (drill 0.4) (layers "F.Cu" "B.Cu") (free) (net 6))
-  (via (at 111.506 88.646) (size 0.8) (drill 0.4) (layers "F.Cu" "B.Cu") (free) (net 6))
-  (via (at 121.412 76.708) (size 0.8) (drill 0.4) (layers "F.Cu" "B.Cu") (free) (net 6))
+  (via (at 118.999 83.439) (size 0.8) (drill 0.4) (layers "F.Cu" "B.Cu") (free) (net 6))
+  (via (at 121.539 74.93) (size 0.8) (drill 0.4) (layers "F.Cu" "B.Cu") (free) (net 6))
+  (via (at 121.031 83.439) (size 0.8) (drill 0.4) (layers "F.Cu" "B.Cu") (free) (net 6))
+  (via (at 121.539 76.962) (size 0.8) (drill 0.4) (layers "F.Cu" "B.Cu") (free) (net 6))
   (segment (start 106.742 90.424) (end 106.742 92.01) (width 0.5) (layer "F.Cu") (net 7))
   (segment (start 106.742 92.01) (end 108.966 94.234) (width 0.5) (layer "F.Cu") (net 7))
@@
   (segment (start 104.202 76.392) (end 104.202 77.724) (width 0.25) (layer "F.Cu") (net 9))
   (segment (start 109.474 77.724) (end 109.474 76.454) (width 0.25) (layer "F.Cu") (net 9))
-  (segment (start 106.742 77.724) (end 107.442 77.724) (width 0.25) (layer "F.Cu") (net 10))
-  (segment (start 110.998 81.28) (end 121.412 81.28) (width 0.25) (layer "F.Cu") (net 10))
-  (segment (start 107.442 77.724) (end 110.998 81.28) (width 0.25) (layer "F.Cu") (net 10))
   (segment (start 123.18 83.048) (end 123.932 83.048) (width 0.25) (layer "F.Cu") (net 10))
+  (segment (start 106.742 77.724) (end 107.823 77.724) (width 0.25) (layer "F.Cu") (net 10))
   (segment (start 121.412 81.28) (end 123.18 83.048) (width 0.25) (layer "F.Cu") (net 10))
-  (segment (start 119.644 85.588) (end 123.932 85.588) (width 0.25) (layer "B.Cu") (net 11))
-  (segment (start 117.094 88.138) (end 119.644 85.588) (width 0.25) (layer "B.Cu") (net 11))
-  (segment (start 101.6 91.694) (end 102.616 92.71) (width 0.25) (layer "B.Cu") (net 11))
-  (segment (start 109.474 92.71) (end 114.046 88.138) (width 0.25) (layer "B.Cu") (net 11))
-  (segment (start 114.046 88.138) (end 117.094 88.138) (width 0.25) (layer "B.Cu") (net 11))
-  (segment (start 102.616 92.71) (end 109.474 92.71) (width 0.25) (layer "B.Cu") (net 11))
-  (segment (start 104.202 85.344) (end 102.616 85.344) (width 0.25) (layer "B.Cu") (net 11))
-  (segment (start 101.6 86.36) (end 101.6 91.694) (width 0.25) (layer "B.Cu") (net 11))
-  (segment (start 102.616 85.344) (end 101.6 86.36) (width 0.25) (layer "B.Cu") (net 11))
+  (segment (start 107.823 77.724) (end 111.379 81.28) (width 0.25) (layer "F.Cu") (net 10))
+  (segment (start 111.379 81.28) (end 121.412 81.28) (width 0.25) (layer "F.Cu") (net 10))
+  (segment (start 102.616 85.344) (end 104.202 85.344) (width 0.25) (layer "B.Cu") (net 11))
+  (segment (start 123.932 85.588) (end 119.644 85.588) (width 0.25) (layer "B.Cu") (net 11))
+  (segment (start 101.6 86.36) (end 102.616 85.344) (width 0.25) (layer "B.Cu") (net 11))
+  (segment (start 102.616 92.71) (end 101.6 91.694) (width 0.25) (layer "B.Cu") (net 11))
+  (segment (start 101.6 91.694) (end 101.6 86.36) (width 0.25) (layer "B.Cu") (net 11))
+  (segment (start 117.094 88.138) (end 113.538 88.138) (width 0.25) (layer "B.Cu") (net 11))
+  (segment (start 119.644 85.588) (end 117.094 88.138) (width 0.25) (layer "B.Cu") (net 11))
+  (segment (start 113.538 88.138) (end 108.966 92.71) (width 0.25) (layer "B.Cu") (net 11))
+  (segment (start 108.966 92.71) (end 102.616 92.71) (width 0.25) (layer "B.Cu") (net 11))
   (segment (start 136.632 80.508) (end 139.202 80.508) (width 1) (layer "F.Cu") (net 12))
   (segment (start 139.202 80.508) (end 143.256 76.454) (width 1) (layer "F.Cu") (net 12))
